Commit message: committing last working torque

File: models/bi_panda/coke.urdf (robot description, URDF)
Before this commit: robot cylinder, 1 links, 0 joints
Links:
- link cylinder: mass 2.5 -> 1; geometry collision cylinder length=0.08 radius=0.015; visual cylinder length=0.08 radius=0.015

Commit message: forces accounting for torque, all planners calculate naive vel and accel

File: models/bi_panda/coke.urdf (robot description, URDF)
Before this commit: robot cylinder, 1 links, 0 joints
Links:
- link cylinder: mass 1 -> 5

Commit message: set up new torque and dynamics fns

File: models/bi_panda/coke.urdf (robot description, URDF)
Before this commit: robot cylinder, 1 links, 0 joints
Links:
- link cylinder: mass 5 -> 100; geometry collision cylinder length=0.05 radius=0.015; visual cylinder length=0.05 radius=0.015

Commit message: rrt* and dynamics updates

File: models/bi_panda/coke.urdf (robot description, URDF)
Before this commit: robot cylinder, 1 links, 0 joints
Links:
- link cylinder: mass 100 -> 7

Commit message: improvements

File: models/bi_panda/coke.urdf (robot description, URDF)
Before this commit: robot cylinder, 1 links, 0 joints
Links:
- link cylinder: mass 7 -> 6

Commit message: anuj rne impl working, min-jerk working

File: models/bi_panda/coke.urdf (robot description, URDF)
Before this commit: robot cylinder, 1 links, 0 joints
Links:
- link cylinder: mass 6 -> 9

File: models/bi_panda/panda.urdf (robot description, URDF)
Before this commit: robot panda, 13 links, 12 joints
Links:
- removed link panda_grasptarget
- link panda_hand: mass .81 -> 0.68; geometry collision mesh filename=meshes/panda/collision/hand.stl; visual mesh filename=meshes/panda/visual/hand.dae
- link panda_leftfinger: mass 0.1 -> 0.01; geometry collision mesh filename=meshes/panda/collision/finger.stl; visual mesh filename=meshes/panda/visual/finger.dae
- link panda_link0: mass 2.9 -> None; geometry collision mesh filename=meshes/panda/collision/link0.stl; visual mesh filename=meshes/panda/visual/link0.dae
- link panda_link1: mass 2.7 -> 4.970684; geometry collision mesh filename=meshes/panda/collision/link1.stl; visual mesh filename=meshes/panda/visual/link1.dae
- link panda_link2: mass 2.73 -> 0.646926; geometry collision mesh filename=meshes/panda/collision/link2.stl; visual mesh filename=meshes/panda/visual/link2.dae
- link panda_link3: mass 2.04 -> 3.228604; geometry collision mesh filename=meshes/panda/collision/link3.stl; visual mesh filename=meshes/panda/visual/link3.dae
- link panda_link4: mass 2.08 -> 3.587895; geometry collision mesh filename=meshes/panda/collision/link4.stl; visual mesh filename=meshes/panda/visual/link4.dae
- link panda_link5: mass 3 -> 1.225946; geometry collision mesh filename=meshes/panda/collision/link5.stl; visual mesh filename=meshes/panda/visual/link5.dae
- link panda_link6: mass 1.3 -> 1.666555; geometry collision mesh filename=meshes/panda/collision/link6.stl; visual mesh filename=meshes/panda/visual/link6.dae
- link panda_link7: mass .2 -> 7.35522e-01; geometry collision mesh filename=meshes/panda/collision/link7.stl; visual mesh filename=meshes/panda/visual/link7.dae
- link panda_rightfinger: mass 0.1 -> 0.01; geometry collision mesh filename=meshes/panda/collision/finger.stl; visual mesh filename=meshes/panda/visual/finger.dae
Joints:
- removed joint panda_grasptarget_hand
- joint panda_finger_joint1: type fixed -> prismatic
- joint panda_finger_joint2: type fixed -> prismatic
- joint panda_joint1: limit lower=-2.9671 upper=2.9671 effort=87 velocity=2.1750 -> lower=-2.8973 upper=2.8973 effort=87 velocity=2.1750
- joint panda_joint2: limit lower=-1.8326 upper=1.8326 effort=87 velocity=2.1750 -> lower=-1.7628 upper=1.7628 effort=87 velocity=2.1750
- joint panda_joint3: limit lower=-2.9671 upper=2.9671 effort=87 velocity=2.1750 -> lower=-2.8973 upper=2.8973 effort=87 velocity=2.1750
- joint panda_joint4: limit lower=-3.1416 upper=0.0 effort=87 velocity=2.1750 -> lower=-3.0718 upper=-0.0698 effort=87 velocity=2.1750
- joint panda_joint5: limit lower=-2.9671 upper=2.9671 effort=12 velocity=2.6100 -> lower=-2.8973 upper=2.8973 effort=12 velocity=2.6100
- joint panda_joint6: limit lower=-0.0873 upper=3.8223 effort=12 velocity=2.6100 -> lower=-0.0175 upper=3.7525 effort=12 velocity=2.6100; origin xyz=0 0 0 rpy=0 0 0 -> xyz=0 0 0 rpy=1.57079632679 0 0
- joint panda_joint7: limit lower=-2.9671 upper=2.9671 effort=12 velocity=2.6100 -> lower=-2.8973 upper=2.8973 effort=12 velocity=2.6100
