Commit message: got hiro sim working

File: models/bi_panda/panda_mod.urdf (robot description, URDF)
Before this commit: robot panda, 13 links, 12 joints
Links:
- removed link r_panda_grasptarget
- removed link r_panda_hand
- removed link r_panda_leftfinger
- removed link r_panda_link0
- removed link r_panda_link1
- removed link r_panda_link2
- removed link r_panda_link3
- removed link r_panda_link4
- removed link r_panda_link5
- removed link r_panda_link6
- removed link r_panda_link7
- removed link r_panda_link8
- removed link r_panda_rightfinger
- added link panda_grasptarget, mass 0.0
- added link panda_hand, mass 0.68; collision mesh filename=meshes/panda/collision/hand.stl; visual mesh filename=meshes/panda/visual/hand.dae
- added link panda_leftfinger, mass 0.01; collision mesh filename=meshes/panda/collision/finger.stl; visual mesh filename=meshes/panda/visual/finger.dae
- added link panda_link0; collision mesh filename=meshes/panda/collision/link0.stl; visual mesh filename=meshes/panda/visual/link0.dae
- added link panda_link1, mass 4.970684; collision mesh filename=meshes/panda/collision/link1.stl; visual mesh filename=meshes/panda/visual/link1.dae
- added link panda_link2, mass 0.646926; collision mesh filename=meshes/panda/collision/link2.stl; visual mesh filename=meshes/panda/visual/link2.dae
- added link panda_link3, mass 3.228604; collision mesh filename=meshes/panda/collision/link3.stl; visual mesh filename=meshes/panda/visual/link3.dae
- added link panda_link4, mass 3.587895; collision mesh filename=meshes/panda/collision/link4.stl; visual mesh filename=meshes/panda/visual/link4.dae
- added link panda_link5, mass 1.225946; collision mesh filename=meshes/panda/collision/link5.stl; visual mesh filename=meshes/panda/visual/link5.dae
- added link panda_link6, mass 1.666555; collision mesh filename=meshes/panda/collision/link6.stl; visual mesh filename=meshes/panda/visual/link6.dae
- added link panda_link7, mass 7.35522e-01; collision mesh filename=meshes/panda/collision/link7.stl; visual mesh filename=meshes/panda/visual/link7.dae
- added link panda_link8, mass 0.0
- added link panda_rightfinger, mass 0.01; collision mesh filename=meshes/panda/collision/finger.stl; visual mesh filename=meshes/panda/visual/finger.dae
Joints:
- removed joint r_panda_finger_joint1
- removed joint r_panda_finger_joint2
- removed joint r_panda_grasptarget_hand
- removed joint r_panda_hand_joint
- removed joint r_panda_joint1
- removed joint r_panda_joint2
- removed joint r_panda_joint3
- removed joint r_panda_joint4
- removed joint r_panda_joint5
- removed joint r_panda_joint6
- removed joint r_panda_joint7
- removed joint r_panda_joint8
- added joint panda_finger_joint1: type prismatic, parent panda_hand, child panda_leftfinger, origin xyz=0 0 0.0584 rpy=0 0 0, axis 0 1 0, limit lower=0.0 upper=0.04 effort=20 velocity=0.2
- added joint panda_finger_joint2: type prismatic, parent panda_hand, child panda_rightfinger, origin xyz=0 0 0.0584 rpy=0 0 0, axis 0 -1 0, limit lower=0.0 upper=0.04 effort=20 velocity=0.2, mimic joint=panda_finger_joint1
- added joint panda_grasptarget_hand: type fixed, parent panda_hand, child panda_grasptarget, origin xyz=0 0 0.105 rpy=0 0 0
- added joint panda_hand_joint: type fixed, parent panda_link8, child panda_hand, origin xyz=0 0 0 rpy=0 0 -0.785398163397
- added joint panda_joint1: type revolute, parent panda_link0, child panda_link1, origin xyz=0 0 0.333 rpy=0 0 0, axis 0 0 1, limit lower=-2.8973 upper=2.8973 effort=87 velocity=2.1750
- added joint panda_joint2: type revolute, parent panda_link1, child panda_link2, origin xyz=0 0 0 rpy=-1.57079632679 0 0, axis 0 0 1, limit lower=-1.7628 upper=1.7628 effort=87 velocity=2.1750
- added joint panda_joint3: type revolute, parent panda_link2, child panda_link3, origin xyz=0 -0.316 0 rpy=1.57079632679 0 0, axis 0 0 1, limit lower=-2.8973 upper=2.8973 effort=87 velocity=2.1750
- added joint panda_joint4: type revolute, parent panda_link3, child panda_link4, origin xyz=0.0825 0 0 rpy=1.57079632679 0 0, axis 0 0 1, limit lower=-3.0718 upper=-0.0698 effort=87 velocity=2.1750
- added joint panda_joint5: type revolute, parent panda_link4, child panda_link5, origin xyz=-0.0825 0.384 0 rpy=-1.57079632679 0 0, axis 0 0 1, limit lower=-2.8973 upper=2.8973 effort=12 velocity=2.6100
- added joint panda_joint6: type revolute, parent panda_link5, child panda_link6, origin xyz=0 0 0 rpy=1.57079632679 0 0, axis 0 0 1, limit lower=-0.0175 upper=3.7525 effort=12 velocity=2.6100
- added joint panda_joint7: type revolute, parent panda_link6, child panda_link7, origin xyz=0.088 0 0 rpy=1.57079632679 0 0, axis 0 0 1, limit lower=-2.8973 upper=2.8973 effort=12 velocity=2.6100
- added joint panda_joint8: type fixed, parent panda_link7, child panda_link8, origin xyz=0 0 0.107 rpy=0 0 0, axis 0 0 0
